Commit message: Revert "Merge branch 'indigo_dev' of https://github.com/ipa-cob4-8/cob_robots into indigo_dev"
This reverts commit 00b785f9b771826134277fd3652434af114bba50, reversing
changes made to 8882110d169ef9126a104a48881272278d5da5f0.

File: cob_hardware_config/robots/cob4-10/urdf/cob4-10.urdf.xacro (robot description, xacro)
@@ -37,5 +37,5 @@
     <origin xyz="${laser_right_x} ${laser_right_y} ${laser_right_z}" rpy="${laser_right_roll} ${laser_right_pitch} ${laser_right_yaw}" />
   </xacro:sick_s300_laser_v0>
-  <xacro:torso name="torso" parent="base_link" dof1="false" dof2="true" dof3="true">
+  <xacro:torso name="torso" parent="base_link" dof1="false" dof2="false" dof3="false">
     <origin xyz="${torso_x} ${torso_y} ${torso_z}" rpy="${torso_roll} ${torso_pitch} ${torso_yaw}" />
   </xacro:torso>
@@ -52,5 +52,5 @@
     <origin xyz="${torso_cam3d_down_x} ${torso_cam3d_down_y} ${torso_cam3d_down_z}" rpy="${torso_cam3d_down_roll} ${torso_cam3d_down_pitch} ${torso_cam3d_down_yaw}" />
   </xacro:realsense>
-  <xacro:head name="head" parent="torso_3_link" dof1="true" dof2="true" dof3="true">
+  <xacro:head name="head" parent="torso_3_link" dof1="false" dof2="false" dof3="false">
     <origin xyz="${head_x} ${head_y} ${head_z}" rpy="${head_roll} ${head_pitch} ${head_yaw}" />
   </xacro:head>

File: cob_hardware_config/robots/cob4-13/urdf/cob4-13.urdf.xacro (robot description, xacro)
@@ -12,7 +12,7 @@
   <xacro:include filename="$(find cob_description)/urdf/cob4_torso/torso.urdf.xacro" />
   <!-- arm -->
-  <xacro:include filename="$(find cob_description)/urdf/cob4_arm/cob4_arm.urdf.xacro" />
+  <!-- xacro:include filename="$(find cob_description)/urdf/cob4_arm/cob4_arm.urdf.xacro" /-->
   <!-- hand -->
-  <xacro:include filename="$(find cob_description)/urdf/cob4_gripper/gripper.urdf.xacro" />
+  <!-- xacro:include filename="$(find cob_description)/urdf/cob4_gripper/gripper.urdf.xacro" /-->
   <!-- head -->
   <xacro:include filename="$(find cob_description)/urdf/cob4_head/head.urdf.xacro" />
@@ -63,15 +63,3 @@
     <origin xyz="${sensorring_cam3d_x} ${sensorring_cam3d_y} ${sensorring_cam3d_z}" rpy="${sensorring_cam3d_roll} ${sensorring_cam3d_pitch} ${sensorring_cam3d_yaw}" />
   </xacro:realsense_zr300>
-  <xacro:cob4_arm name="arm_right" parent="torso_3_link" has_podest="false">
-    <origin xyz="${arm_right_x} ${arm_right_y} ${arm_right_z}" rpy="${arm_right_roll} ${arm_right_pitch} ${arm_right_yaw}" />
-  </xacro:cob4_arm>
-  <xacro:cob4_arm name="arm_left" parent="torso_3_link" has_podest="false">
-    <origin xyz="${arm_left_x} ${arm_left_y} ${arm_left_z}" rpy="${arm_left_roll} ${arm_left_pitch} ${arm_left_yaw}" />
-  </xacro:cob4_arm>
-  <xacro:gripper name="gripper_right" parent="arm_right_7_link">
-    <origin xyz="${gripper_right_x} ${gripper_right_y} ${gripper_right_z}" rpy="${gripper_right_roll} ${gripper_right_pitch} ${gripper_right_yaw}" />
-  </xacro:gripper>
-  <xacro:gripper name="gripper_left" parent="arm_left_7_link">
-    <origin xyz="${gripper_left_x} ${gripper_left_y} ${gripper_left_z}" rpy="${gripper_left_roll} ${gripper_left_pitch} ${gripper_left_yaw}" />
-  </xacro:gripper>
 </robot>

File: cob_hardware_config/robots/cob4-7/urdf/calibration_default.urdf.xacro (robot description, xacro)
@@ -63,36 +63,37 @@
 	<xacro:property name="def_arm_left_pitch" value="0"/>
 	<xacro:property name="def_arm_left_yaw" value="3.14159"/>
-	<!-- ***************************** -->
-	<!-- extrinsic camera calibration  -->
-	<!-- ***************************** -->
-	<!-- torso cam3d left mount positions | relative to torso_3_link -->
-	<xacro:property name="def_torso_cam3d_left_x" value="0.14873"/>
-	<xacro:property name="def_torso_cam3d_left_y" value="0.01293"/>
-	<xacro:property name="def_torso_cam3d_left_z" value="0.27008"/>
-	<xacro:property name="def_torso_cam3d_left_roll" value="-1.57079"/>
+	<!-- *********************************** -->
+	<!-- kinematic chain reference positions -->
+	<!-- *********************************** -->
+	<!-- this feature is no longer supported as urdfdom does not parse the according 'calibration_rising' tag -->
+	<!-- cam3d left | handeye calibration | relative to torso_3_link -->
+	<xacro:property name="def_torso_cam3d_left_x" value="0.12839"/>
+	<xacro:property name="def_torso_cam3d_left_y" value="0.01802"/>
+	<xacro:property name="def_torso_cam3d_left_z" value="0.24214"/>
+	<xacro:property name="def_torso_cam3d_left_roll" value="1.57079"/>
 	<xacro:property name="def_torso_cam3d_left_pitch" value="0.0"/>
-	<xacro:property name="def_torso_cam3d_left_yaw" value="0.61"/>
-	<!-- torso cam3d right mount positions | relative to torso_3_link -->
-	<xacro:property name="def_torso_cam3d_right_x" value="0.14873"/>
-	<xacro:property name="def_torso_cam3d_right_y" value="-0.01293"/>
-	<xacro:property name="def_torso_cam3d_right_z" value="0.27008"/>
-	<xacro:property name="def_torso_cam3d_right_roll" value="-1.57079"/>
+	<xacro:property name="def_torso_cam3d_left_yaw" value="0.418879"/>
+	<!-- cam3d right | handeye calibration | relative to torso_3_link -->
+	<xacro:property name="def_torso_cam3d_right_x" value="0.12839"/>
+	<xacro:property name="def_torso_cam3d_right_y" value="-0.01802"/>
+	<xacro:property name="def_torso_cam3d_right_z" value="0.24214"/>
+	<xacro:property name="def_torso_cam3d_right_roll" value="1.57079"/>
 	<xacro:property name="def_torso_cam3d_right_pitch" value="0.0"/>
-	<xacro:property name="def_torso_cam3d_right_yaw" value="-0.61"/>
-	<!-- torso cam3d down mount positions | relative to torso_3_link -->
-	<xacro:property name="def_torso_cam3d_down_x" value="0.15203"/>
+	<xacro:property name="def_torso_cam3d_right_yaw" value="-0.418879"/>
+	<!-- cam3d down | handeye calibration | relative to torso_3_link -->
+	<xacro:property name="def_torso_cam3d_down_x" value="0.15908"/>
 	<xacro:property name="def_torso_cam3d_down_y" value="0.0"/>
-	<xacro:property name="def_torso_cam3d_down_z" value="0.1307"/>
+	<xacro:property name="def_torso_cam3d_down_z" value="0.14005"/>
 	<xacro:property name="def_torso_cam3d_down_roll" value="0.0"/>
-	<xacro:property name="def_torso_cam3d_down_pitch" value="0.56"/>
+	<xacro:property name="def_torso_cam3d_down_pitch" value="0.61086"/>
 	<xacro:property name="def_torso_cam3d_down_yaw" value="0.0"/>
-	<!-- sensorring cam3d mount positions | relative to sensorring_link -->
-	<xacro:property name="def_sensorring_cam3d_x" value="0.1251"/>
+	<!-- cam3d | handeye calibration | relative to sensorring_link -->
+	<xacro:property name="def_sensorring_cam3d_x" value="0.096"/>
 	<xacro:property name="def_sensorring_cam3d_y" value="0.0"/>
-	<xacro:property name="def_sensorring_cam3d_z" value="0.001"/>
+	<xacro:property name="def_sensorring_cam3d_z" value="0.0195"/>
 	<xacro:property name="def_sensorring_cam3d_roll" value="0.0"/>
 	<xacro:property name="def_sensorring_cam3d_pitch" value="0.0"/>
 	<xacro:property name="def_sensorring_cam3d_yaw" value="0.0"/>
-	<!-- head cam mount positions | relative to head_3_link -->
+	<!-- cam | handeye calibration | relative to head_3_link -->
 	<xacro:property name="def_head_cam_x" value="-0.181"/>
 	<xacro:property name="def_head_cam_y" value="0.0"/>

File: cob_hardware_config/robots/cob4-7/urdf/cob4-7.urdf.xacro (robot description, xacro)
@@ -64,5 +64,5 @@
     <origin xyz="${arm_left_x} ${arm_left_y} ${arm_left_z}" rpy="${arm_left_roll} ${arm_left_pitch} ${arm_left_yaw}" />
   </xacro:cob4_arm>
-  <xacro:sensorring name="sensorring" parent="head_3_link" active="true">
+  <xacro:sensorring name="sensorring" parent="head_3_link" active="false">  <!-- HotFix: set active to true when the HW is repaired -->
     <origin xyz="${sensorring_x} ${sensorring_y} ${sensorring_z}" rpy="${sensorring_roll} ${sensorring_pitch} ${sensorring_yaw}" />
   </xacro:sensorring>
